File: Resources/Electronics/Kaffettino/Kaffettino.kicad_sch (KiCad schematic)
At the start: 48 parts, among them J1 PPTC101LFBN-RC, J2 OSTVN02A150, J3 OSTVN02A150, J4 OSTVN02A150, J5 OSTVN02A150, M1 RFID-RC522, U1 PCF8574AN, U2 ESP32-38Pin-Wroom, U3 DFR0299

Commit message: Corrected some footprints in the PCB schema
Parts:
- removed J3, J4, J5: OSTVN02A150, OSTVN02A150:CONN_OSTVN02A150_OST, symbol 2025-11-11_16-38-17:OSTVN02A150
- added H1, H2, H3, H4: MountingHole, MountingHole:MountingHole_3.2mm_M3, symbol Mechanical:MountingHole
- added J3, J5: OSTVN04A150, OSTVN04A150:CONN_OSTVN04A150_OST, symbol 2025-11-13_14-58-24:OSTVN04A150
- added R24: 10k, Resistor_THT:R_Axial_DIN0207_L6.3mm_D2.5mm_P10.16mm_Horizontal, symbol Device:R
- D1, D2, D3: footprint LED_THT:LED_D3.0mm -> LED_THT:LED_D5.0mm
Connections:
- net +3.3V: now also J3.1, J5.1, R24.2
- net EXPANSION_1: now also J3.2
- net EXPANSION_2: now also J3.3
- net GEN_SCL: now also J5.2
- net GEN_SDA: now also J5.3
- net GNDREF: now also J3.4, J5.4
- net RFID_INT: now also R24.1
Other:
- note added: "EXPANSION I2C"
- note removed: "EXPANSION PIN I2C"
- moved on the sheet: BZ1, C10, J2, LS1, M1, R12, R13, R14, R23, U3
