File: Resources/Electronics/Kaffettino/Kaffettino.kicad_pcb (KiCad board)
At the start: 2 copper layers, 150 x 150 mm, 68 parts, among them J1 OSTVN05A150, J2 OSTVN02A150, J3 OSTVN05A150, J5 OSTVN04A150, M1 RFID-RC522, Q1 PN2222A, U1 PCF8574AN, U2 DFR0299, U3 ESP32-38Pin-Wroom, U4 26052

Commit message: Fixed wrong PCB label 3.3 to 5V
Parts:
- removed kibuzzard-69A1ABE5: G***, kibuzzard-69A1ABE5
- added kibuzzard-69A86FC7: G***, kibuzzard-69A86FC7, F.Cu at (60.7, 154.6)
